File: hardware/mainboard/mainboard/mainboard.kicad_sch (KiCad schematic)
At the start: 0 parts

Commit message: hardware(mainboard): complete schematic + first-pass PCB layout
Parts:
- added A2: IMU, Connector_PinSocket_2.54mm:PinSocket_1x05_P2.54mm_Vertical, symbol Connector_Generic:Conn_01x05
- added A3: MP1584, mainboard:MP1584_Module, symbol Connector_Generic:Conn_01x04
- added C1: 470uF/35V, Capacitor_THT:CP_Radial_D8.0mm_P3.50mm, symbol Device:C_Polarized
- added C10: 1uF, Capacitor_THT:C_Disc_D5.0mm_W2.5mm_P5.00mm, symbol Device:C
- added C2: 100uF/16V, Capacitor_THT:CP_Radial_D6.3mm_P2.50mm, symbol Device:C_Polarized
- added C3, C4, C5, C7: 100nF, Capacitor_THT:C_Disc_D5.0mm_W2.5mm_P5.00mm, symbol Device:C
- added D1: SMBJ24A, Diode_SMD:D_SMB, symbol Device:D_Zener
- added D3: SMBJ20A, Diode_SMD:D_SMB, symbol Device:D_Zener
- added Dz1: 18V, Diode_THT:D_DO-35_SOD27_P7.62mm_Horizontal, symbol Device:D_Zener
- added J1, J5: (no value), TerminalBlock:TerminalBlock_MaiXu_MX126-5.0-02P_1x02_P5.00mm, symbol Connector_Generic:Conn_01x02
- added J2: Conn_01x02, TerminalBlock:TerminalBlock_MaiXu_MX126-5.0-02P_1x02_P5.00mm, symbol Connector_Generic:Conn_01x02
- added J3: Conn_01x04, TerminalBlock:TerminalBlock_MaiXu_MX126-5.0-04P_1x04_P5.00mm, symbol Connector_Generic:Conn_01x04
- added J4: (no value), TerminalBlock:TerminalBlock_MaiXu_MX126-5.0-03P_1x03_P5.00mm, symbol Connector_Generic:Conn_01x03
- added J6: (no value), Connector_PinHeader_2.54mm:PinHeader_1x04_P2.54mm_Vertical, symbol Connector_Generic:Conn_01x04
- added J8, J9: ESP32, Connector_PinSocket_2.54mm:PinSocket_1x19_P2.54mm_Vertical, symbol Connector_Generic:Conn_01x19
- added Q1: AOD4185, Package_TO_SOT_THT:TO-220-3_Vertical, symbol Transistor_FET:Q_PMOS_GSD
- added R1, R10, R2, R3, R4, R9: 10k, Resistor_THT:R_Axial_DIN0207_L6.3mm_D2.5mm_P7.62mm_Horizontal, symbol Device:R
- added R11: 100k, Resistor_THT:R_Axial_DIN0207_L6.3mm_D2.5mm_P7.62mm_Horizontal, symbol Device:R
- added R12, R14: 100, Resistor_THT:R_Axial_DIN0207_L6.3mm_D2.5mm_P7.62mm_Horizontal, symbol Device:R
- added R5, R6: 4.7k, Resistor_THT:R_Axial_DIN0207_L6.3mm_D2.5mm_P7.62mm_Horizontal, symbol Device:R
- added R7, R8: 2.2k, Resistor_THT:R_Axial_DIN0207_L6.3mm_D2.5mm_P7.62mm_Horizontal, symbol Device:R
- added U2: ULN2803A, Package_DIP:DIP-18_W7.62mm_Socket, symbol Transistor_Array:ULN2803A
- added U3: INA3221, Connector_PinSocket_2.54mm:PinSocket_1x06_P2.54mm_Vertical, symbol Connector_Generic:Conn_01x06
- added U4, U5: PC817, Package_DIP:DIP-4_W7.62mm, symbol Isolator:PC817
Connections:
- new net: R7.2, U4.1
- new net: C10.1, D3.1 (K), R14.2
- new net: R8.2, U5.1
- new net: Dz1.2 (A), Q1.1 (G), R11.2, R12.2
- new net +12V_HOT: J1.1 (Pin_1), Q1.3 (D)
- new net +12V_PROT: A3.1 (Pin_1), C1.1, D1.1 (K), Dz1.1 (K), Q1.2 (S), R11.1
- new net +3.3V: A2.3 (Pin_3), C3.1, C5.2, C7.1, J6.1 (Pin_1), J8.1 (Pin_1), R10.2, R5.1, R6.1, R9.2, U3.1 (Pin_1)
- new net +5V: A3.3 (Pin_3), C2.1, J8.19 (Pin_19)
- new net COIL_FOG: J3.2 (Pin_2), U2.17 (O2)
- new net COIL_GRIP: J3.3 (Pin_3), U2.16 (O3)
- new net COIL_MASTER: J3.1 (Pin_1), U2.18 (O1)
- new net COIL_RAIL: C4.1, J2.1 (Pin_1), U2.10 (COM)
- new net COIL_SPARE: J3.4 (Pin_4), U2.15 (O4)
- new net FOG_EN: J8.9 (Pin_9), R2.1, U2.2 (I2)
- new net GND: A2.4 (Pin_4), A3.2 (Pin_2), A3.4 (Pin_4), C1.2, C10.2, C2.2, C3.2, C4.2, C5.1, C7.2, D1.2 (A), D3.2 (A), J1.2 (Pin_2), J2.2 (Pin_2), J4.3 (Pin_3), J5.2 (Pin_2), J6.4 (Pin_4), J9.1 (Pin_1), J9.7 (Pin_7), R1.2, R12.1, R2.2, R3.2, R4.2, U2.5 (I5), U2.6 (I6), U2.7 (I7), U2.8 (I8), U2.9 (GND), U3.2 (Pin_2), U4.2, U4.3, U5.2, U5.3
- new net GRIP_EN: J8.10 (Pin_10), R3.1, U2.3 (I3)
- new net IGN_12V: J4.1 (Pin_1), R7.1
- new net IGN_SENSE: J8.5 (Pin_5), R9.1, U4.4
- new net IMU_INT: A2.5 (Pin_5), J8.8 (Pin_8)
- new net MASTER_EN: J8.15 (Pin_15), R1.1, U2.1 (I1)
- new net SCL: A2.2 (Pin_2), J6.3 (Pin_3), J9.3 (Pin_3), R6.2, U3.4 (Pin_4)
- new net SDA: A2.1 (Pin_1), J6.2 (Pin_2), J9.6 (Pin_6), R5.2, U3.3 (Pin_3)
- new net SENSE: U3.5 (Pin_5), U3.6 (Pin_6)
- new net SPARE_EN: J8.11 (Pin_11), R4.1, U2.4 (I4)
- new net START_12V: J4.2 (Pin_2), R8.1
- new net START_SENSE: J8.6 (Pin_6), R10.1, U5.4
- new net VBUS_SENSE: J5.1 (Pin_1), R14.1
